File: hardware/source_trigger_unit/flyback.kicad_sch (KiCad schematic)
At the start: 26 parts, among them Q1 STF10N60M2, T1 D-120W-S20, T3 Transformer_1P_1S, U6 LM317_TO-220, U7 1ED3124MU12F

Commit message: add titles & reformat schematics
Other:
- company: (none) -> Dawson HEP
- title: (none) -> Flyback Converter (STU)
Changed lines of the file:
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@@
 	(generator_version "9.0")
 	(paper "A4")
+	(title_block
+		(title "Flyback Converter (STU)")
+		(date "2026-03-09")
+		(rev "V1")
+		(company "Dawson HEP")
+		(comment 1 "Alex Xia")
+	)
 	(circle
 		(center 192.405 95.25)
