File: hardware/source_trigger_unit/power.kicad_sch (KiCad schematic)
At the start: 21 parts, among them K2 12V, M3 Fan, M4 Fan, T5 N-68X, 120V-120V 50VA

Commit message: add titles & reformat schematics
Other:
- company: (none) -> Dawson HEP
- title: (none) -> Power Supply (STU)
Changed lines of the file:
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@@
 	(generator_version "9.0")
 	(paper "A4")
+	(title_block
+		(title "Power Supply (STU)")
+		(date "2026-03-09")
+		(rev "V1")
+		(company "Dawson HEP")
+		(comment 1 "Alex Xia")
+	)
 	(rectangle
 		(start 81.915 36.83)
