File: hardware/source_trigger_unit/spark_chamber.kicad_sch (KiCad schematic)
At the start: 8 parts

Commit message: add titles & reformat schematics
Other:
- company: (none) -> Dawson HEP
- title: (none) -> Spark Chamber
Changed lines of the file:
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@@
 	(generator_version "9.0")
 	(paper "A4")
+	(title_block
+		(title "Spark Chamber")
+		(date "2026-03-09")
+		(rev "V1")
+		(company "Dawson HEP")
+		(comment 1 "Alex Xia")
+	)
 	(bezier
 		(pts
