File: hardware/source_trigger_unit/trigger_spark_gap.kicad_sch (KiCad schematic)
At the start: 15 parts, among them Q2 STF10N60M2, T4 ZS1052, TRIGGER COIL, U5 1ED3124MU12F

Commit message: add titles & reformat schematics
Other:
- company: (none) -> Dawson HEP
- title: (none) -> Spark Gap Trigger (STU)
Changed lines of the file:
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@@
 	(generator_version "9.0")
 	(paper "A4")
+	(title_block
+		(title "Spark Gap Trigger (STU)")
+		(date "2026-03-09")
+		(rev "V1")
+		(company "Dawson HEP")
+		(comment 1 "Alex Xia")
+	)
 	(text "GALVANIC ISOLATION\n3.0 kV_{RMS}\n200 kV/us CMTI"
 		(exclude_from_sim no)
